File: scratch-rp2040-60p.kicad_sch (KiCad schematic)
At the start: 29 parts, among them P1 USB_C_Plug_USB2.0, SW1 SW_Push, SW1 SW_SPST, U1 RP2040, U2 NCP1117-3.3_SOT223, U3 W25Q128JVS, Y1 12MHz

Commit message: footprint assigned
Parts:
- added D10, D11, D12, D13, D14, D15, D16, D17, D18, D19, D2, D20, D21, D22, D23, D24, D25, D26, D27, D28, D29, D3, D30, D31, D32, D33, D34, D35, D36, D37, D38, D39, D4, D40, D41, D42, D43, D44, D45, D46, D47, D48, D49, D5, D50, D51, D52, D53, D54, D55, D56, D57, D58, D59, D6, D60, D61, D7, D8, D9: 1N4148W, Diode_SMD:D_SOD-523, symbol Diode:1N4148W
- added LED10, LED11, LED12, LED13, LED14, LED15, LED16, LED17, LED18, LED19, LED2, LED20, LED21, LED22, LED23, LED24, LED25, LED26, LED27, LED28, LED29, LED3, LED30, LED31, LED32, LED33, LED34, LED35, LED36, LED37, LED38, LED39, LED4, LED40, LED41, LED42, LED43, LED44, LED45, LED46, LED47, LED48, LED49, LED5, LED50, LED51, LED52, LED53, LED54, LED55, LED56, LED57, LED58, LED59, LED6, LED61, LED63, LED7, LED8, LED9: LED_SK6812MINI-E, LED_SMD:LED_SK6812_PLCC4_5.0x5.0mm_P3.2mm, symbol LED:SK6812
- added SW10, SW11, SW12, SW13, SW16, SW17, SW18, SW19, SW2, SW20, SW21, SW22, SW23, SW24, SW25, SW26, SW27, SW3, SW30, SW31, SW32, SW33, SW34, SW35, SW36, SW37, SW38, SW39, SW4, SW40, SW43, SW44, SW45, SW46, SW47, SW48, SW49, SW5, SW50, SW51, SW52, SW6, SW7, SW8, SW9: SW_Push, kbd_SW:CherryMX_Hotswap_1u, symbol Switch:SW_Push
- added SW14: SW_Push, kbd_SW:CherryMX_Hotswap_2u, symbol Switch:SW_Push
- added SW15, SW28: SW_Push, kbd_SW:CherryMX_Hotswap_1.5u, symbol Switch:SW_Push
- added SW29: SW_Push, kbd_SW:CherryMX_Hotswap_1.75u, symbol Switch:SW_Push
- added SW41, SW42: SW_Push, kbd_SW:CherryMX_Hotswap_2.25u, symbol Switch:SW_Push
- added SW53: SW_Push, kbd_SW:CherryMX_Hotswap_2.75u, symbol Switch:SW_Push
- added SW54, SW55, SW56, SW58, SW59, SW60, SW61: SW_Push, kbd_SW:CherryMX_Hotswap_1.25u, symbol Switch:SW_Push
- added SW57: SW_Push, kbd_SW:CherryMX_Hotswap_6.25u, symbol Switch:SW_Push
- D1: footprint Diode_SMD:D_SOD-123 -> Diode_SMD:D_SOD-523
- LED1: footprint (none) -> LED_SMD:LED_SK6812_PLCC4_5.0x5.0mm_P3.2mm; symbol Salicylic_kbd:LED_SK6812MINI-E -> LED:SK6812
- SW1: footprint (none) -> kbd_SW:CherryMX_Hotswap_1u
Connections:
- net +3.3V: now also LED1.3 (VDD), LED10.3 (VDD), LED11.3 (VDD), LED12.3 (VDD), LED13.3 (VDD), LED14.3 (VDD), LED15.3 (VDD), LED16.3 (VDD), LED17.3 (VDD), LED18.3 (VDD), LED19.3 (VDD), LED2.3 (VDD), LED20.3 (VDD), LED21.3 (VDD), LED22.3 (VDD), LED23.3 (VDD), LED24.3 (VDD), LED25.3 (VDD), LED26.3 (VDD), LED27.3 (VDD), LED28.3 (VDD), LED29.3 (VDD), LED3.3 (VDD), LED30.3 (VDD), LED31.3 (VDD), LED32.3 (VDD), LED33.3 (VDD), LED34.3 (VDD), LED35.3 (VDD), LED36.3 (VDD), LED37.3 (VDD), LED38.3 (VDD), LED39.3 (VDD), LED4.3 (VDD), LED40.3 (VDD), LED41.3 (VDD), LED42.3 (VDD), LED43.3 (VDD), LED44.3 (VDD), LED45.3 (VDD), LED46.3 (VDD), LED47.3 (VDD), LED48.3 (VDD), LED49.3 (VDD), LED5.3 (VDD), LED50.3 (VDD), LED51.3 (VDD), LED52.3 (VDD), LED53.3 (VDD), LED54.3 (VDD), LED55.3 (VDD), LED56.3 (VDD), LED57.3 (VDD), LED58.3 (VDD), LED59.3 (VDD), LED6.3 (VDD), LED61.3 (VDD), LED63.3 (VDD), LED7.3 (VDD), LED8.3 (VDD), LED9.3 (VDD)
- net GND: now also LED1.1 (VSS), LED10.1 (VSS), LED11.1 (VSS), LED12.1 (VSS), LED13.1 (VSS), LED14.1 (VSS), LED15.1 (VSS), LED16.1 (VSS), LED17.1 (VSS), LED18.1 (VSS), LED19.1 (VSS), LED2.1 (VSS), LED20.1 (VSS), LED21.1 (VSS), LED22.1 (VSS), LED23.1 (VSS), LED24.1 (VSS), LED25.1 (VSS), LED26.1 (VSS), LED27.1 (VSS), LED28.1 (VSS), LED29.1 (VSS), LED3.1 (VSS), LED30.1 (VSS), LED31.1 (VSS), LED32.1 (VSS), LED33.1 (VSS), LED34.1 (VSS), LED35.1 (VSS), LED36.1 (VSS), LED37.1 (VSS), LED38.1 (VSS), LED39.1 (VSS), LED4.1 (VSS), LED40.1 (VSS), LED41.1 (VSS), LED42.1 (VSS), LED43.1 (VSS), LED44.1 (VSS), LED45.1 (VSS), LED46.1 (VSS), LED47.1 (VSS), LED48.1 (VSS), LED49.1 (VSS), LED5.1 (VSS), LED50.1 (VSS), LED51.1 (VSS), LED52.1 (VSS), LED53.1 (VSS), LED54.1 (VSS), LED55.1 (VSS), LED56.1 (VSS), LED57.1 (VSS), LED58.1 (VSS), LED59.1 (VSS), LED6.1 (VSS), LED61.1 (VSS), LED63.1 (VSS), LED7.1 (VSS), LED8.1 (VSS), LED9.1 (VSS)
- net at D1.1 (K): now also SW1.2
- net ROW1: now reaches D1.2 (A)
- net ROW1: now also U1.18 (GPIO15), D10.2 (A), D11.2 (A), D12.2 (A), D13.2 (A), D14.2 (A), D2.2 (A), D3.2 (A), D4.2 (A), D5.2 (A), D6.2 (A), D7.2 (A), D8.2 (A), D9.2 (A)
- net LED_IN: now reaches LED1.2 (DIN)
- net LED_IN: now also U1.38 (GPIO26_ADC0)
- net at LED1.4 (DOUT): now also LED2.2 (DIN)
- net COL8: now reaches U1.11 (GPIO8)
- net COL8: now also SW22.1, SW36.1, SW49.1, SW61.1, SW8.1
- net COL9: now reaches U1.12 (GPIO9)
- net COL9: now also SW23.1, SW37.1, SW50.1, SW9.1
- net COL10: now reaches U1.13 (GPIO10)
- net COL10: now also SW10.1, SW24.1, SW38.1, SW51.1
- net COL11: now reaches U1.14 (GPIO11)
- net COL11: now also SW11.1, SW25.1, SW39.1, SW52.1
- net COL12: now reaches U1.15 (GPIO12)
- net COL12: now also SW12.1, SW26.1, SW40.1, SW53.1
- net COL13: now reaches U1.16 (GPIO13)
- net COL13: now also SW13.1, SW27.1, SW41.1
- net COL14: now reaches U1.17 (GPIO14)
- net COL14: now also SW14.1, SW28.1
- net ROW2: now reaches U1.27 (GPIO16)
- net ROW2: now also D15.2 (A), D16.2 (A), D17.2 (A), D18.2 (A), D19.2 (A), D20.2 (A), D21.2 (A), D22.2 (A), D23.2 (A), D24.2 (A), D25.2 (A), D26.2 (A), D27.2 (A), D28.2 (A)
- net ROW3: now reaches U1.28 (GPIO17)
- net ROW3: now also D29.2 (A), D30.2 (A), D31.2 (A), D32.2 (A), D33.2 (A), D34.2 (A), D35.2 (A), D36.2 (A), D37.2 (A), D38.2 (A), D39.2 (A), D40.2 (A), D41.2 (A)
- net ROW4: now reaches U1.29 (GPIO18)
- net ROW4: now also D42.2 (A), D43.2 (A), D44.2 (A), D45.2 (A), D46.2 (A), D47.2 (A), D48.2 (A), D49.2 (A), D50.2 (A), D51.2 (A), D52.2 (A), D53.2 (A)
- net COL1: now reaches U1.3 (GPIO1)
- net COL1: now also SW1.1, SW15.1, SW29.1, SW42.1, SW54.1
- net ROW5: now reaches U1.30 (GPIO19)
- net ROW5: now also D54.2 (A), D55.2 (A), D56.2 (A), D57.2 (A), D58.2 (A), D59.2 (A), D60.2 (A), D61.2 (A)
- net LED_OUT: now reaches U1.39 (GPIO27_ADC1)
- net LED_OUT: now also LED58.4 (DOUT)
- net COL2: now reaches U1.4 (GPIO2)
- net COL2: now also SW16.1, SW2.1, SW30.1, SW43.1, SW55.1
- net COL3: now reaches U1.5 (GPIO3)
- net COL3: now also SW17.1, SW3.1, SW31.1, SW44.1, SW56.1
- net COL4: now reaches U1.6 (GPIO4)
- net COL4: now also SW18.1, SW32.1, SW4.1, SW45.1, SW57.1
- net COL5: now reaches U1.7 (GPIO5)
- net COL5: now also SW19.1, SW33.1, SW46.1, SW5.1, SW58.1
- net COL6: now reaches U1.8 (GPIO6)
- net COL6: now also SW20.1, SW34.1, SW47.1, SW59.1, SW6.1
- net COL7: now reaches U1.9 (GPIO7)
- net COL7: now also SW21.1, SW35.1, SW48.1, SW60.1, SW7.1
- new net: D44.1 (K), SW44.2
- new net: D2.1 (K), SW2.2
- new net: D39.1 (K), SW39.2
- new net: D7.1 (K), SW7.2
- new net: D18.1 (K), SW18.2
- new net: LED41.4 (DOUT), LED43.2 (DIN)
- new net: LED43.4 (DOUT), LED45.2 (DIN)
- new net: D31.1 (K), SW31.2
- new net: LED37.4 (DOUT), LED39.2 (DIN)
- new net: LED39.4 (DOUT), LED41.2 (DIN)
- new net: D9.1 (K), SW9.2
- new net: D16.1 (K), SW16.2
- new net: D28.1 (K), SW28.2
- new net: D8.1 (K), SW8.2
- new net: D34.1 (K), SW34.2
- new net: D24.1 (K), SW24.2
- new net: D46.1 (K), SW46.2
- new net: D13.1 (K), SW13.2
- new net: LED3.4 (DOUT), LED4.2 (DIN)
- new net: LED4.4 (DOUT), LED5.2 (DIN)
- new net: D57.1 (K), SW57.2
- new net: D22.1 (K), SW22.2
- new net: D53.1 (K), SW53.2
- new net: D41.1 (K), SW41.2
- new net: D56.1 (K), SW56.2
- new net: LED32.4 (DOUT), LED33.2 (DIN)
- new net: LED33.4 (DOUT), LED35.2 (DIN)
- new net: D59.1 (K), SW59.2
- new net: LED19.4 (DOUT), LED20.2 (DIN)
- new net: LED20.4 (DOUT), LED21.2 (DIN)
- new net: D5.1 (K), SW5.2
- new net: D43.1 (K), SW43.2
- new net: D3.1 (K), SW3.2
- new net: D15.1 (K), SW15.2
- new net: D12.1 (K), SW12.2
- new net: D42.1 (K), SW42.2
- new net: LED44.4 (DOUT), LED46.2 (DIN)
- new net: LED46.4 (DOUT), LED48.2 (DIN)
- new net: D19.1 (K), SW19.2
- new net: D4.1 (K), SW4.2
- new net: D27.1 (K), SW27.2
- new net: D26.1 (K), SW26.2
- new net: D14.1 (K), SW14.2
- new net: D10.1 (K), SW10.2
- new net: D30.1 (K), SW30.2
- new net: LED21.4 (DOUT), LED22.2 (DIN)
- new net: LED54.4 (DOUT), LED56.2 (DIN)
- new net: LED56.4 (DOUT), LED58.2 (DIN)
- new net: D40.1 (K), SW40.2
- new net: LED35.4 (DOUT), LED37.2 (DIN)
- new net: LED6.4 (DOUT), LED7.2 (DIN)
- new net: LED7.4 (DOUT), LED8.2 (DIN)
- new net: D23.1 (K), SW23.2
- new net: LED15.4 (DOUT), LED16.2 (DIN)
- new net: LED16.4 (DOUT), LED17.2 (DIN)
- new net: D6.1 (K), SW6.2
- new net: LED22.4 (DOUT), LED23.2 (DIN)
- new net: LED23.4 (DOUT), LED24.2 (DIN)
- new net: D32.1 (K), SW32.2
- new net: D52.1 (K), SW52.2
- new net: D21.1 (K), SW21.2
- new net: D51.1 (K), SW51.2
- new net: LED53.4 (DOUT), LED55.2 (DIN)
- new net: LED55.4 (DOUT), LED57.2 (DIN)
- new net: D58.1 (K), SW58.2
- new net: D37.1 (K), SW37.2
- new net: D45.1 (K), SW45.2
- new net: LED17.4 (DOUT), LED18.2 (DIN)
- new net: LED18.4 (DOUT), LED19.2 (DIN)
- new net: D29.1 (K), SW29.2
- new net: D38.1 (K), SW38.2
- new net: LED8.4 (DOUT), LED9.2 (DIN)
- new net: LED10.2 (DIN), LED9.4 (DOUT)
- new net: LED57.4 (DOUT), LED59.2 (DIN)
- new net: LED2.4 (DOUT), LED3.2 (DIN)
- new net: LED29.4 (DOUT), LED30.2 (DIN)
- new net: LED30.4 (DOUT), LED31.2 (DIN)
- new net: LED48.4 (DOUT), LED50.2 (DIN)
- new net: LED50.4 (DOUT), LED52.2 (DIN)
- new net: LED34.4 (DOUT), LED36.2 (DIN)
- new net: LED36.4 (DOUT), LED38.2 (DIN)
- new net: D48.1 (K), SW48.2
- new net: D20.1 (K), SW20.2
- new net: LED47.4 (DOUT), LED49.2 (DIN)
- new net: LED49.4 (DOUT), LED51.2 (DIN)
- new net: LED24.4 (DOUT), LED25.2 (DIN)
- new net: LED45.4 (DOUT), LED47.2 (DIN)
- new net: D50.1 (K), SW50.2
- new net: LED25.4 (DOUT), LED26.2 (DIN)
- new net: D25.1 (K), SW25.2
- new net: LED10.4 (DOUT), LED11.2 (DIN)
- new net: LED11.4 (DOUT), LED12.2 (DIN)
- new net: LED31.4 (DOUT), LED32.2 (DIN)
- new net: LED59.4 (DOUT), LED61.2 (DIN)
- new net: LED61.4 (DOUT), LED63.2 (DIN)
- new net: D11.1 (K), SW11.2
- new net: D17.1 (K), SW17.2
- new net: LED52.4 (DOUT), LED54.2 (DIN)
- new net: D35.1 (K), SW35.2
- new net: LED34.2 (DIN), LED63.4 (DOUT)
- new net: D47.1 (K), SW47.2
- new net: LED51.4 (DOUT), LED53.2 (DIN)
- new net: D36.1 (K), SW36.2
- new net: D54.1 (K), SW54.2
- new net: D61.1 (K), SW61.2
- new net: LED40.4 (DOUT), LED42.2 (DIN)
- new net: LED42.4 (DOUT), LED44.2 (DIN)
- new net: D60.1 (K), SW60.2
- new net: D33.1 (K), SW33.2
- new net: LED26.4 (DOUT), LED27.2 (DIN)
- new net: D55.1 (K), SW55.2
- new net: LED14.4 (DOUT), LED15.2 (DIN)
- new net: LED27.4 (DOUT), LED28.2 (DIN)
- new net: LED28.4 (DOUT), LED29.2 (DIN)
- new net: LED38.4 (DOUT), LED40.2 (DIN)
- new net: D49.1 (K), SW49.2
- new net: LED5.4 (DOUT), LED6.2 (DIN)
- new net: LED12.4 (DOUT), LED13.2 (DIN)
- new net: LED13.4 (DOUT), LED14.2 (DIN)
- no-connect marks 28 -> 13
Other:
- moved on the sheet: D1, SW1

Commit message: 20230922 end
Parts:
- added LED62, LED63: LED_SK6812MINI-E, LED_SMD:LED_SK6812_EC15_1.5x1.5mm, symbol LED:SK6812MINI
- LED1, LED10, LED11, LED12, LED13, LED14, LED15, LED16, LED17, LED18, LED19, LED2, LED20, LED21, LED22, LED23, LED24, LED25, LED26, LED27, LED28, LED29, LED3, LED30, LED31, LED32, LED33, LED4, LED5, LED6, LED7, LED8, LED9: footprint LED_SMD:LED_SK6812_PLCC4_5.0x5.0mm_P3.2mm -> LED_SMD:LED_SK6812_EC15_1.5x1.5mm; symbol LED:SK6812 -> LED:SK6812MINI
- LED34: renamed from LED35; footprint LED_SMD:LED_SK6812_PLCC4_5.0x5.0mm_P3.2mm -> LED_SMD:LED_SK6812_EC15_1.5x1.5mm; symbol LED:SK6812 -> LED:SK6812MINI
- LED35: renamed from LED37; footprint LED_SMD:LED_SK6812_PLCC4_5.0x5.0mm_P3.2mm -> LED_SMD:LED_SK6812_EC15_1.5x1.5mm; symbol LED:SK6812 -> LED:SK6812MINI
- LED36: renamed from LED39; footprint LED_SMD:LED_SK6812_PLCC4_5.0x5.0mm_P3.2mm -> LED_SMD:LED_SK6812_EC15_1.5x1.5mm; symbol LED:SK6812 -> LED:SK6812MINI
- LED37: renamed from LED41; footprint LED_SMD:LED_SK6812_PLCC4_5.0x5.0mm_P3.2mm -> LED_SMD:LED_SK6812_EC15_1.5x1.5mm; symbol LED:SK6812 -> LED:SK6812MINI
- LED38: renamed from LED43; footprint LED_SMD:LED_SK6812_PLCC4_5.0x5.0mm_P3.2mm -> LED_SMD:LED_SK6812_EC15_1.5x1.5mm; symbol LED:SK6812 -> LED:SK6812MINI
- LED39: renamed from LED45; footprint LED_SMD:LED_SK6812_PLCC4_5.0x5.0mm_P3.2mm -> LED_SMD:LED_SK6812_EC15_1.5x1.5mm; symbol LED:SK6812 -> LED:SK6812MINI
- LED40: renamed from LED47; footprint LED_SMD:LED_SK6812_PLCC4_5.0x5.0mm_P3.2mm -> LED_SMD:LED_SK6812_EC15_1.5x1.5mm; symbol LED:SK6812 -> LED:SK6812MINI
- LED41: renamed from LED49; footprint LED_SMD:LED_SK6812_PLCC4_5.0x5.0mm_P3.2mm -> LED_SMD:LED_SK6812_EC15_1.5x1.5mm; symbol LED:SK6812 -> LED:SK6812MINI
- LED42: renamed from LED51; footprint LED_SMD:LED_SK6812_PLCC4_5.0x5.0mm_P3.2mm -> LED_SMD:LED_SK6812_EC15_1.5x1.5mm; symbol LED:SK6812 -> LED:SK6812MINI
- LED43: renamed from LED53; footprint LED_SMD:LED_SK6812_PLCC4_5.0x5.0mm_P3.2mm -> LED_SMD:LED_SK6812_EC15_1.5x1.5mm; symbol LED:SK6812 -> LED:SK6812MINI
- LED44: renamed from LED55; footprint LED_SMD:LED_SK6812_PLCC4_5.0x5.0mm_P3.2mm -> LED_SMD:LED_SK6812_EC15_1.5x1.5mm; symbol LED:SK6812 -> LED:SK6812MINI
- LED45: renamed from LED57; footprint LED_SMD:LED_SK6812_PLCC4_5.0x5.0mm_P3.2mm -> LED_SMD:LED_SK6812_EC15_1.5x1.5mm; symbol LED:SK6812 -> LED:SK6812MINI
- LED46: renamed from LED59; footprint LED_SMD:LED_SK6812_PLCC4_5.0x5.0mm_P3.2mm -> LED_SMD:LED_SK6812_EC15_1.5x1.5mm; symbol LED:SK6812 -> LED:SK6812MINI
- LED47: renamed from LED61; footprint LED_SMD:LED_SK6812_PLCC4_5.0x5.0mm_P3.2mm -> LED_SMD:LED_SK6812_EC15_1.5x1.5mm; symbol LED:SK6812 -> LED:SK6812MINI
- LED48: renamed from LED63; footprint LED_SMD:LED_SK6812_PLCC4_5.0x5.0mm_P3.2mm -> LED_SMD:LED_SK6812_EC15_1.5x1.5mm; symbol LED:SK6812 -> LED:SK6812MINI
- LED49: renamed from LED34; footprint LED_SMD:LED_SK6812_PLCC4_5.0x5.0mm_P3.2mm -> LED_SMD:LED_SK6812_EC15_1.5x1.5mm; symbol LED:SK6812 -> LED:SK6812MINI
- LED50: renamed from LED36; footprint LED_SMD:LED_SK6812_PLCC4_5.0x5.0mm_P3.2mm -> LED_SMD:LED_SK6812_EC15_1.5x1.5mm; symbol LED:SK6812 -> LED:SK6812MINI
- LED51: renamed from LED38; footprint LED_SMD:LED_SK6812_PLCC4_5.0x5.0mm_P3.2mm -> LED_SMD:LED_SK6812_EC15_1.5x1.5mm; symbol LED:SK6812 -> LED:SK6812MINI
- LED52: renamed from LED40; footprint LED_SMD:LED_SK6812_PLCC4_5.0x5.0mm_P3.2mm -> LED_SMD:LED_SK6812_EC15_1.5x1.5mm; symbol LED:SK6812 -> LED:SK6812MINI
- LED53: renamed from LED42; footprint LED_SMD:LED_SK6812_PLCC4_5.0x5.0mm_P3.2mm -> LED_SMD:LED_SK6812_EC15_1.5x1.5mm; symbol LED:SK6812 -> LED:SK6812MINI
- LED54: renamed from LED44; footprint LED_SMD:LED_SK6812_PLCC4_5.0x5.0mm_P3.2mm -> LED_SMD:LED_SK6812_EC15_1.5x1.5mm; symbol LED:SK6812 -> LED:SK6812MINI
- LED55: renamed from LED46; footprint LED_SMD:LED_SK6812_PLCC4_5.0x5.0mm_P3.2mm -> LED_SMD:LED_SK6812_EC15_1.5x1.5mm; symbol LED:SK6812 -> LED:SK6812MINI
- LED56: renamed from LED48; footprint LED_SMD:LED_SK6812_PLCC4_5.0x5.0mm_P3.2mm -> LED_SMD:LED_SK6812_EC15_1.5x1.5mm; symbol LED:SK6812 -> LED:SK6812MINI
- LED57: renamed from LED50; footprint LED_SMD:LED_SK6812_PLCC4_5.0x5.0mm_P3.2mm -> LED_SMD:LED_SK6812_EC15_1.5x1.5mm; symbol LED:SK6812 -> LED:SK6812MINI
- LED58: renamed from LED52; footprint LED_SMD:LED_SK6812_PLCC4_5.0x5.0mm_P3.2mm -> LED_SMD:LED_SK6812_EC15_1.5x1.5mm; symbol LED:SK6812 -> LED:SK6812MINI
- LED59: renamed from LED54; footprint LED_SMD:LED_SK6812_PLCC4_5.0x5.0mm_P3.2mm -> LED_SMD:LED_SK6812_EC15_1.5x1.5mm; symbol LED:SK6812 -> LED:SK6812MINI
- LED60: renamed from LED56; footprint LED_SMD:LED_SK6812_PLCC4_5.0x5.0mm_P3.2mm -> LED_SMD:LED_SK6812_EC15_1.5x1.5mm; symbol LED:SK6812 -> LED:SK6812MINI
- LED61: renamed from LED58; footprint LED_SMD:LED_SK6812_PLCC4_5.0x5.0mm_P3.2mm -> LED_SMD:LED_SK6812_EC15_1.5x1.5mm; symbol LED:SK6812 -> LED:SK6812MINI
Connections:
- net +3.3V: now also LED1.4 (VDD), LED10.4 (VDD), LED11.4 (VDD), LED12.4 (VDD), LED13.4 (VDD), LED14.4 (VDD), LED15.4 (VDD), LED16.4 (VDD), LED17.4 (VDD), LED18.4 (VDD), LED19.4 (VDD), LED2.4 (VDD), LED20.4 (VDD), LED21.4 (VDD), LED22.4 (VDD), LED23.4 (VDD), LED24.4 (VDD), LED25.4 (VDD), LED26.4 (VDD), LED27.4 (VDD), LED28.4 (VDD), LED29.4 (VDD), LED3.4 (VDD), LED30.4 (VDD), LED31.4 (VDD), LED32.4 (VDD), LED33.4 (VDD), LED34.4 (VDD), LED35.4 (VDD), LED36.4 (VDD), LED37.4 (VDD), LED38.4 (VDD), LED39.4 (VDD), LED4.4 (VDD), LED40.4 (VDD), LED41.4 (VDD), LED42.4 (VDD), LED43.4 (VDD), LED44.4 (VDD), LED45.4 (VDD), LED46.4 (VDD), LED47.4 (VDD), LED48.4 (VDD), LED49.4 (VDD), LED5.4 (VDD), LED50.4 (VDD), LED51.4 (VDD), LED52.4 (VDD), LED53.4 (VDD), LED54.4 (VDD), LED55.4 (VDD), LED56.4 (VDD), LED57.4 (VDD), LED58.4 (VDD), LED59.4 (VDD), LED6.4 (VDD), LED60.4 (VDD), LED61.4 (VDD), LED7.4 (VDD), LED8.4 (VDD), LED9.4 (VDD), LED62.4 (VDD), LED63.4 (VDD); no longer LED1.3 (VDD), LED10.3 (VDD), LED11.3 (VDD), LED12.3 (VDD), LED13.3 (VDD), LED14.3 (VDD), LED15.3 (VDD), LED16.3 (VDD), LED17.3 (VDD), LED18.3 (VDD), LED19.3 (VDD), LED2.3 (VDD), LED20.3 (VDD), LED21.3 (VDD), LED22.3 (VDD), LED23.3 (VDD), LED24.3 (VDD), LED25.3 (VDD), LED26.3 (VDD), LED27.3 (VDD), LED28.3 (VDD), LED29.3 (VDD), LED3.3 (VDD), LED30.3 (VDD), LED31.3 (VDD), LED32.3 (VDD), LED33.3 (VDD), LED34.3 (VDD), LED35.3 (VDD), LED36.3 (VDD), LED37.3 (VDD), LED38.3 (VDD), LED39.3 (VDD), LED4.3 (VDD), LED40.3 (VDD), LED41.3 (VDD), LED42.3 (VDD), LED43.3 (VDD), LED44.3 (VDD), LED45.3 (VDD), LED46.3 (VDD), LED47.3 (VDD), LED48.3 (VDD), LED49.3 (VDD), LED5.3 (VDD), LED50.3 (VDD), LED51.3 (VDD), LED52.3 (VDD), LED53.3 (VDD), LED54.3 (VDD), LED55.3 (VDD), LED56.3 (VDD), LED57.3 (VDD), LED58.3 (VDD), LED59.3 (VDD), LED6.3 (VDD), LED60.3 (VDD), LED61.3 (VDD), LED7.3 (VDD), LED8.3 (VDD), LED9.3 (VDD)
- net GND: now also LED1.2 (VSS), LED10.2 (VSS), LED11.2 (VSS), LED12.2 (VSS), LED13.2 (VSS), LED14.2 (VSS), LED15.2 (VSS), LED16.2 (VSS), LED17.2 (VSS), LED18.2 (VSS), LED19.2 (VSS), LED2.2 (VSS), LED20.2 (VSS), LED21.2 (VSS), LED22.2 (VSS), LED23.2 (VSS), LED24.2 (VSS), LED25.2 (VSS), LED26.2 (VSS), LED27.2 (VSS), LED28.2 (VSS), LED29.2 (VSS), LED3.2 (VSS), LED30.2 (VSS), LED31.2 (VSS), LED32.2 (VSS), LED33.2 (VSS), LED34.2 (VSS), LED35.2 (VSS), LED36.2 (VSS), LED37.2 (VSS), LED38.2 (VSS), LED39.2 (VSS), LED4.2 (VSS), LED40.2 (VSS), LED41.2 (VSS), LED42.2 (VSS), LED43.2 (VSS), LED44.2 (VSS), LED45.2 (VSS), LED46.2 (VSS), LED47.2 (VSS), LED48.2 (VSS), LED49.2 (VSS), LED5.2 (VSS), LED50.2 (VSS), LED51.2 (VSS), LED52.2 (VSS), LED53.2 (VSS), LED54.2 (VSS), LED55.2 (VSS), LED56.2 (VSS), LED57.2 (VSS), LED58.2 (VSS), LED59.2 (VSS), LED6.2 (VSS), LED60.2 (VSS), LED61.2 (VSS), LED7.2 (VSS), LED8.2 (VSS), LED9.2 (VSS), LED62.2 (VSS), LED63.2 (VSS); no longer LED1.1 (VSS), LED10.1 (VSS), LED11.1 (VSS), LED12.1 (VSS), LED13.1 (VSS), LED14.1 (VSS), LED15.1 (VSS), LED16.1 (VSS), LED17.1 (VSS), LED18.1 (VSS), LED19.1 (VSS), LED2.1 (VSS), LED20.1 (VSS), LED21.1 (VSS), LED22.1 (VSS), LED23.1 (VSS), LED24.1 (VSS), LED25.1 (VSS), LED26.1 (VSS), LED27.1 (VSS), LED28.1 (VSS), LED29.1 (VSS), LED3.1 (VSS), LED30.1 (VSS), LED31.1 (VSS), LED32.1 (VSS), LED33.1 (VSS), LED34.1 (VSS), LED35.1 (VSS), LED36.1 (VSS), LED37.1 (VSS), LED38.1 (VSS), LED39.1 (VSS), LED4.1 (VSS), LED40.1 (VSS), LED41.1 (VSS), LED42.1 (VSS), LED43.1 (VSS), LED44.1 (VSS), LED45.1 (VSS), LED46.1 (VSS), LED47.1 (VSS), LED48.1 (VSS), LED49.1 (VSS), LED5.1 (VSS), LED50.1 (VSS), LED51.1 (VSS), LED52.1 (VSS), LED53.1 (VSS), LED54.1 (VSS), LED55.1 (VSS), LED56.1 (VSS), LED57.1 (VSS), LED58.1 (VSS), LED59.1 (VSS), LED6.1 (VSS), LED60.1 (VSS), LED61.1 (VSS), LED7.1 (VSS), LED8.1 (VSS), LED9.1 (VSS)
- net LED_IN: now also LED1.3 (DIN); no longer LED1.2 (DIN)
- net LED_OUT: now also LED63.1 (DOUT); no longer LED61.4 (DOUT)
- new net: LED38.1 (DOUT), LED39.3 (DIN)
- new net: LED37.1 (DOUT), LED38.3 (DIN)
- new net: LED62.1 (DOUT), LED63.3 (DIN)
- new net: LED36.1 (DOUT), LED37.3 (DIN)
- new net: LED35.1 (DOUT), LED36.3 (DIN)
- new net: LED4.1 (DOUT), LED5.3 (DIN)
- new net: LED3.1 (DOUT), LED4.3 (DIN)
- new net: LED33.1 (DOUT), LED34.3 (DIN)
- new net: LED32.1 (DOUT), LED33.3 (DIN)
- new net: LED20.1 (DOUT), LED21.3 (DIN)
- new net: LED19.1 (DOUT), LED20.3 (DIN)
- new net: LED61.1 (DOUT), LED62.3 (DIN)
- new net: LED55.1 (DOUT), LED56.3 (DIN)
- new net: LED54.1 (DOUT), LED55.3 (DIN)
- new net: LED21.1 (DOUT), LED22.3 (DIN)
- new net: LED60.1 (DOUT), LED61.3 (DIN)
- new net: LED59.1 (DOUT), LED60.3 (DIN)
- new net: LED34.1 (DOUT), LED35.3 (DIN)
- new net: LED7.1 (DOUT), LED8.3 (DIN)
- new net: LED6.1 (DOUT), LED7.3 (DIN)
- new net: LED16.1 (DOUT), LED17.3 (DIN)
- new net: LED15.1 (DOUT), LED16.3 (DIN)
- new net: LED23.1 (DOUT), LED24.3 (DIN)
- new net: LED22.1 (DOUT), LED23.3 (DIN)
- new net: LED44.1 (DOUT), LED45.3 (DIN)
- new net: LED43.1 (DOUT), LED44.3 (DIN)
- new net: LED17.1 (DOUT), LED18.3 (DIN)
- new net: LED1.1 (DOUT), LED2.3 (DIN)
- new net: LED18.1 (DOUT), LED19.3 (DIN)
- new net: LED10.3 (DIN), LED9.1 (DOUT)
- new net: LED8.1 (DOUT), LED9.3 (DIN)
- new net: LED45.1 (DOUT), LED46.3 (DIN)
- new net: LED2.1 (DOUT), LED3.3 (DIN)
- new net: LED30.1 (DOUT), LED31.3 (DIN)
- new net: LED29.1 (DOUT), LED30.3 (DIN)
- new net: LED57.1 (DOUT), LED58.3 (DIN)
- new net: LED56.1 (DOUT), LED57.3 (DIN)
- new net: LED50.1 (DOUT), LED51.3 (DIN)
- new net: LED49.1 (DOUT), LED50.3 (DIN)
- new net: LED41.1 (DOUT), LED42.3 (DIN)
- new net: LED40.1 (DOUT), LED41.3 (DIN)
- new net: LED24.1 (DOUT), LED25.3 (DIN)
- new net: LED39.1 (DOUT), LED40.3 (DIN)
- new net: LED25.1 (DOUT), LED26.3 (DIN)
- new net: LED11.1 (DOUT), LED12.3 (DIN)
- new net: LED10.1 (DOUT), LED11.3 (DIN)
- new net: LED31.1 (DOUT), LED32.3 (DIN)
- new net: LED47.1 (DOUT), LED48.3 (DIN)
- new net: LED46.1 (DOUT), LED47.3 (DIN)
- new net: LED58.1 (DOUT), LED59.3 (DIN)
- new net: LED48.1 (DOUT), LED49.3 (DIN)
- new net: LED42.1 (DOUT), LED43.3 (DIN)
- new net: LED53.1 (DOUT), LED54.3 (DIN)
- new net: LED52.1 (DOUT), LED53.3 (DIN)
- new net: LED26.1 (DOUT), LED27.3 (DIN)
- new net: LED14.1 (DOUT), LED15.3 (DIN)
- new net: LED27.1 (DOUT), LED28.3 (DIN)
- new net: LED28.1 (DOUT), LED29.3 (DIN)
- new net: LED51.1 (DOUT), LED52.3 (DIN)
- new net: LED5.1 (DOUT), LED6.3 (DIN)
- new net: LED13.1 (DOUT), LED14.3 (DIN)
- new net: LED12.1 (DOUT), LED13.3 (DIN)
