File: scratch-rp2040-60p.kicad_pcb (KiCad board)
At the start: 2 copper layers, 211 parts, among them P1 USB_C_Plug_USB2.0, SW1 SW_Push, SW10 SW_Push, SW11 SW_Push, SW12 SW_Push, SW13 SW_Push, SW14 SW_Push, SW15 SW_Push, SW16 SW_Push, SW17 SW_Push, SW18 SW_Push, SW19 SW_Push, SW2 SW_Push, SW20 SW_Push, SW21 SW_Push, SW22 SW_Push, SW23 SW_Push, SW24 SW_Push, SW25 SW_Push, SW26 SW_Push, SW27 SW_Push, SW28 SW_Push, SW29 SW_Push, SW3 SW_Push, SW30 SW_Push, SW31 SW_Push, SW32 SW_Push, SW33 SW_Push, SW34 SW_Push, SW35 SW_Push, SW36 SW_Push, SW37 SW_Push, SW38 SW_Push, SW39 SW_Push, SW4 SW_Push, SW40 SW_Push, SW41 SW_Push, SW42 SW_Push, SW43 SW_Push, SW44 SW_Push, SW45 SW_Push, SW46 SW_Push, SW47 SW_Push, SW48 SW_Push, SW49 SW_Push, SW5 SW_Push, SW50 SW_Push, SW51 SW_Push, SW52 SW_Push, SW53 SW_Push, SW54 SW_Push, SW55 SW_Push, SW56 SW_Push, SW57 SW_Push, SW58 SW_Push, SW59 SW_Push, SW6 SW_Push, SW60 SW_Push, SW61 SW_Push, SW62 SW_SPST, SW7 SW_Push, SW8 SW_Push, SW9 SW_Push, U1 W25Q128JVS, U2 RP2040, U3 NCP1117-3.3_SOT223, Y1 12MHz

Commit message: commit
Parts:
- moved U1 93.1 mm to (210.8, 71.9)
- moved C3 79.7 mm to (120.6, 133.3)
- moved Y1 78.9 mm to (122.7, 137.3)
- moved U2 75.6 mm to (121.6, 127.5)
- moved SW62 73.7 mm to (163.0, 77.0)
- moved U3 54.3 mm to (139.7, 78.6)
- moved P1 25.5 mm to (109.5, 79.7), turned to 180 degrees
- moved C1 20.2 mm to (123.9, 62.2)
- moved C10 20.2 mm to (126.3, 65.7)
- moved C11 20.2 mm to (126.3, 67.4)
- moved C12 20.2 mm to (126.3, 69.2)
- moved C13 20.2 mm to (126.3, 70.9)
- moved C14 20.2 mm to (119.6, 71.7)
- moved C15 20.2 mm to (126.3, 72.7)
- moved C16 20.2 mm to (119.6, 73.7)
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
Commit message: commit
Parts:
- turned LED15 to 90 degrees
Routing:
- net GND: track 0.00 -> 139.3 mm
- net +3.3V: track 0.00 -> 136.1 mm, vias 0 -> 13
- net Net-(LED13-DOUT): track 0.00 -> 28.0 mm, vias 0 -> 2
- net Net-(LED14-DOUT): track 0.00 -> 22.4 mm
- net Net-(LED3-DOUT): track 0.00 -> 18.5 mm, vias 0 -> 2
- net Net-(LED5-DOUT): track 0.00 -> 18.5 mm, vias 0 -> 2
- net Net-(LED7-DOUT): track 0.00 -> 18.5 mm, vias 0 -> 2
- net Net-(LED11-DOUT): track 0.00 -> 18.5 mm, vias 0 -> 2
- net Net-(LED1-DOUT): track 0.00 -> 18.5 mm, vias 0 -> 2
- net Net-(LED10-DIN): track 0.00 -> 18.5 mm, vias 0 -> 2
- net Net-(LED4-DOUT): track 0.00 -> 18.5 mm
- net Net-(LED2-DOUT): track 0.00 -> 18.5 mm
- net Net-(LED10-DOUT): track 0.00 -> 18.5 mm
- net Net-(LED8-DOUT): track 0.00 -> 18.5 mm
- net Net-(LED6-DOUT): track 0.00 -> 18.5 mm
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